Commit message: Fixed .dae model path

File: rb1_base_description/urdf/custom_stuff/custom_stuff.urdf.xacro (robot description, xacro)
@@ -30,5 +30,5 @@
             <geometry>
                 <!--box size=".4 .2 .1"/-->
-                <mesh filename = "package://biscee_simulation/meshes/biscee.dae"/>
+                <mesh filename = "package://rb1_base_description/urdf/biscee/biscee.dae"/>
                 <!--cylinder length="1.0" radius="0.20" /-->
             </geometry>

Commit message: Added urdf for camera

File: rb1_base_description/urdf/custom_stuff/custom_stuff.urdf.xacro (robot description, xacro)
@@ -30,5 +30,5 @@
             <geometry>
                 <!--box size=".4 .2 .1"/-->
-                <mesh filename = "package://rb1_base_description/urdf/biscee/biscee.dae"/>
+                <mesh filename="package://rb1_base_description/urdf/biscee/biscee.dae" />
                 <!--cylinder length="1.0" radius="0.20" /-->
             </geometry>
@@ -36,4 +36,6 @@
         </visual>
     </link>
+    <!-- Camera (does not work under Virtualbox -->
+    <!-- xacro:include filename="$(find rb1_base_description)/urdf/custom_stuff/camera_with_base.urdf.xacro"/-->
     <joint name="uh_front_joint" type="fixed">
         <axis xyz="0 1 0" />
